Commit message: M2.8: dual-arm handover pipeline — 12DOF OMPL planning + servo lifecycle fix
DualMoveToJointState:
- new DualMoveToJointState.action interface (12 joint goal)
- new dual_move_server: /plan_kinematic_path (dual_arm group) →
  split trajectory → send to both controllers directly
- motion_nodes: DualMoveToJointState BT wrapper

Servo lifecycle fix (servo ↔ trajectory conflict):
- ServoLifecycleManager: add force_start() (bypass state cache)
- move_to_pose_server: stop_servo → force_stop
- visual_align_server: start_servo → force_start
- dual_move_server: unconditional force_stop both arms before plan

Other fixes:
- s622_dual_arm.launch.py: add fairino_ik_service (/fairino/get_all_ik)
- scene_nodes: fix TransferObject registered as DetachObjectNode
- bt_dual_config.yaml: dual_home + dual_handover_ready named poses
- pick_handover_place.xml: full handover BT tree
- arm_actions_dual.launch.py: dual launch with left/right/dual namespaces

Co-Authored-By: Claude <noreply@anthropic.com>

File: src/gz_launch/config/robot_gazebo.urdf.xacro (robot description, xacro)
@@ -2,13 +2,22 @@
 <robot xmlns:xacro="http://www.ros.org/wiki/xacro" name="s622">
     <xacro:property name="M_PI" value="3.1415926535897931" />
-    <xacro:arg
-        name="initial_positions_file"
-        default="$(find s622_moveit_config)/config/initial_positions.yaml" />
+    <!-- ============ 参数声明 ============ -->
+    <xacro:arg name="robot_name" default="s622"/>
+    <xacro:arg name="prefix" default=""/>
+    <xacro:arg name="attach_world" default="true"/>
+    <xacro:arg name="include_camera" default="true"/>
+    <xacro:arg name="controllers_yaml"
+               default="$(find s622_moveit_config)/config/ros2_controllers.yaml"/>
+    <xacro:arg name="initial_positions_file"
+               default="$(find s622_moveit_config)/config/initial_positions.yaml" />
+    <xacro:property name="prefix" value="$(arg prefix)"/>
+    <!-- ============ 引入本体 URDF (xacro) ============ -->
     <xacro:include
-        filename="$(find s622_moveit_descriptions)/urdf/s622_moveit_descriptions.urdf" />
+        filename="$(find s622_moveit_descriptions)/urdf/s622_moveit_descriptions.urdf.xacro" />
+    <!-- ============ Gazebo 全局插件 ============ -->
     <gazebo>
         <plugin filename="gz_ros2_control-system"
             name="gz_ros2_control::GazeboSimROS2ControlPlugin">
-            <parameters>$(find s622_moveit_config)/config/ros2_controllers.yaml</parameters>
+            <parameters>$(arg controllers_yaml)</parameters>
         </plugin>
         <plugin filename="gz-sim-joint-state-publisher-system"
@@ -25,26 +34,6 @@
         </plugin>
     </gazebo>
-    <!-- <gazebo reference="camera_link">
-        <sensor name="rgbd_camera" type="rgbd_camera">
-            <update_rate>30</update_rate>
-            <topic>camera</topic>
-            <camera>
-        <horizontal_fov>1.047</horizontal_fov>
-        <image>
-            <width>640</width>
-            <height>480</height>
-        </image>
-        <clip>
-            <near>0.05</near>
-            <far>5.0</far>
-        </clip>
-    </camera>
-            <always_on>1</always_on>
-            <visualize>true</visualize>
-        </sensor>
-    </gazebo>
-    -->
-    <!-- 夹爪摩擦参数（防 Gazebo 抖动） -->
-    <gazebo reference="finger1_joint">
+    <!-- ============ 夹爪摩擦 (前缀化) ============ -->
+    <gazebo reference="${prefix}finger1_joint">
         <mu1>500.0</mu1>
         <mu2>500.0</mu2>
@@ -52,5 +41,5 @@
         <kd>15</kd>
     </gazebo>
-    <gazebo reference="finger2_joint">
+    <gazebo reference="${prefix}finger2_joint">
         <mu1>500.0</mu1>
         <mu2>500.0</mu2>
@@ -58,23 +47,19 @@
         <kd>15</kd>
     </gazebo>
-    <!-- ros2_control 标签实例化 -->
-    <!-- <xacro:include filename="$(find
-    s622_moveit_config)/config/s622_moveit_descriptions.ros2_control.xacro"/>
-    <xacro:s622_moveit_descriptions_ros2_control
-        name="GazeboSimSystem"
-        initial_positions_file="$(arg initial_positions_file)"/> -->
+    <!-- ============ ros2_control 实例化 ============ -->
     <xacro:include
         filename="$(find gz_launch)/config/s622_gazebo_ros2_control.xacro" />
     <xacro:s622_moveit_descriptions_ros2_control
         name="GazeboSimSystem"
-        initial_positions_file="$(arg initial_positions_file)" />
-    <!-- Camera -->
-    <xacro:include
-        filename="$(find s622_moveit_descriptions)/urdf/camera/camera.xacro" />
-    <xacro:camera_v0
-        parent="base_link">
-        <!-- A: 右侧俯视工作区中心 (0.35, 0, 0.10) -->
-        <origin xyz="0.35 0.5 0.9" rpy="0 ${58*M_PI/180} ${-M_PI/2}"/>
-    </xacro:camera_v0>
-    <xacro:camera_gazebo_v0 />
+        initial_positions_file="$(arg initial_positions_file)"
+        prefix="${prefix}" />
+    <!-- ============ Camera (可选) ============ -->
+    <xacro:if value="$(arg include_camera)">
+        <xacro:include
+            filename="$(find s622_moveit_descriptions)/urdf/camera/camera.xacro" />
+        <xacro:camera_v0 parent="${prefix}base_link">
+            <origin xyz="0.35 0.5 0.9" rpy="0 ${58*M_PI/180} ${-M_PI/2}"/>
+        </xacro:camera_v0>
+        <xacro:camera_gazebo_v0 />
+    </xacro:if>
 </robot>

File: src/gz_launch/config/s622_gazebo_ros2_control.xacro (robot description, xacro)
@@ -1,13 +1,15 @@
 <?xml version="1.0"?>
 <robot xmlns:xacro="http://www.ros.org/wiki/xacro">
+    <!-- 增加 prefix 参数, 默认为空以保持 M1.7 兼容 -->
     <xacro:macro name="s622_moveit_descriptions_ros2_control"
-        params="name initial_positions_file">
+        params="name initial_positions_file prefix:=''">
         <xacro:property name="initial_positions"
             value="${load_yaml(initial_positions_file)['initial_positions']}" />
-        <ros2_control name="${name}" type="system">
+        <ros2_control name="${prefix}${name}" type="system">
             <hardware>
                 <plugin>gz_ros2_control/GazeboSimSystem</plugin>
             </hardware>
-            <joint name="j1">
+            <!-- 6 个关节全部前缀化,同时 initial_positions 用无前缀 key 索引 -->
+            <joint name="${prefix}j1">
                 <command_interface name="velocity" />
                 <state_interface name="position">
@@ -16,5 +18,5 @@
                 <state_interface name="velocity" />
             </joint>
-            <joint name="j2">
+            <joint name="${prefix}j2">
                 <command_interface name="velocity" />
                 <state_interface name="position">
@@ -23,5 +25,5 @@
                 <state_interface name="velocity" />
             </joint>
-            <joint name="j3">
+            <joint name="${prefix}j3">
                 <command_interface name="velocity" />
                 <state_interface name="position">
@@ -30,5 +32,5 @@
                 <state_interface name="velocity" />
             </joint>
-            <joint name="j4">
+            <joint name="${prefix}j4">
                 <command_interface name="velocity" />
                 <state_interface name="position">
@@ -37,5 +39,5 @@
                 <state_interface name="velocity" />
             </joint>
-            <joint name="j5">
+            <joint name="${prefix}j5">
                 <command_interface name="velocity" />
                 <state_interface name="position">
@@ -44,5 +46,5 @@
                 <state_interface name="velocity" />
             </joint>
-            <joint name="j6">
+            <joint name="${prefix}j6">
                 <command_interface name="velocity" />
                 <state_interface name="position">
@@ -51,17 +53,15 @@
                 <state_interface name="velocity" />
             </joint>
-            <joint name="finger1_joint">
+            <joint name="${prefix}finger1_joint">
                 <command_interface name="position" />
                 <state_interface name="position">
                     <param name="initial_value">${initial_positions['finger1_joint']}</param>
                 </state_interface>
-                <!-- <state_interface name="velocity"/> -->
             </joint>
-            <joint name="finger2_joint">
+            <joint name="${prefix}finger2_joint">
                 <command_interface name="position" />
                 <state_interface name="position">
                     <param name="initial_value">${initial_positions['finger2_joint']}</param>
                 </state_interface>
-                <!-- <state_interface name="velocity"/> -->
             </joint>
         </ros2_control>
