Commit message: chore: misc fixes (camera intrinsics, servo config, table launch cleanup)
杂项历史遗留（2026-08-25 整理提交）：
- camera.xacro/rgbd_split.gazebo.xacro: hfov 82.4° 内参修复（gz rgbd 分离）
- robot_gazebo.urdf.xacro: 相机/模型配置更新
- s622_table.launch.py: 移除 fairino_ik_service（已并入 FairinoIKPlugin）
- servo.yaml: 参数更新
- s622_dual_arm.urdf.xacro / s622_dual_arm_gazebo.urdf.xacro: 双臂 xacro 修正
- gz_launch/CMakeLists.txt: 清理
- .gitignore: 排除 *.tar.gz / .codegraph/ / tmp/
- .claude/settings.json: s622_embodied 权限
- 新增 test_single_arm.launch.py / s622_world.sdf

File: src/gz_launch/config/robot_gazebo.urdf.xacro (robot description, xacro)
@@ -7,4 +7,5 @@
     <xacro:arg name="attach_world" default="true"/>
     <xacro:arg name="include_camera" default="true"/>
+    <xacro:arg name="include_camera_visual" default="false"/>  <!-- false=简化几何体，RViz 不卡 -->
     <xacro:arg name="controllers_yaml"
                default="$(find s622_moveit_config)/config/ros2_controllers.yaml"/>
@@ -15,4 +16,8 @@
     <xacro:include
         filename="$(find s622_moveit_descriptions)/urdf/s622_moveit_descriptions.urdf.xacro" />
+    <!-- ============ 显式实例化机械臂本体 ============
+         M2.8 后主 xacro 的 instantiate 默认改为 false（供双臂顶层显式实例化），
+         单臂顶层需显式调用 s622_arm 一次（与 s622_dual_arm_gazebo.urdf.xacro 风格一致） -->
+    <xacro:s622_arm prefix="$(arg prefix)" attach_world="$(arg attach_world)" />
     <!-- ============ Gazebo 全局插件 ============ -->
     <gazebo>
@@ -55,8 +60,10 @@
         prefix="${prefix}" />
     <!-- ============ Camera (可选) ============ -->
+    <!-- include_camera_visual: false(默认)=简化几何体，RViz 不卡；true=真实 mesh -->
     <xacro:if value="$(arg include_camera)">
         <xacro:include
             filename="$(find s622_moveit_descriptions)/urdf/camera/camera.xacro" />
-        <xacro:camera_v0 parent="${prefix}base_link">
+        <xacro:camera_v0 parent="${prefix}base_link"
+                         use_camera_visual="$(arg include_camera_visual)">
             <origin xyz="0.35 0.5 0.9" rpy="0 ${58*M_PI/180} ${-M_PI/2}"/>
         </xacro:camera_v0>

File: src/gz_launch/config/s622_dual_arm_gazebo.urdf.xacro (robot description, xacro)
@@ -2,5 +2,5 @@
 <robot xmlns:xacro="http://www.ros.org/wiki/xacro" name="s622_dual_arm">
     <xacro:property name="M_PI" value="3.14159265358979323846" />
-    <xacro:arg name="instantiate" default="false"/>   <!-- ← 加这行 -->
+    <xacro:arg name="instantiate" default="false" />   <!-- ← 加这行 -->
     <!-- ============ world 根 link ============ -->
     <link name="world" />
@@ -27,4 +27,5 @@
     <xacro:include
         filename="$(find s622_moveit_descriptions)/urdf/s622_moveit_descriptions.urdf.xacro" />
+    <xacro:property name="instantiate" value="false" />
     <!-- ============ Left Arm: (0.35, 0, 0), yaw=π ============ -->
     <xacro:s622_arm prefix="left_" attach_world="false" />

File: src/s622_moveit_config/config/s622_dual_arm.urdf.xacro (robot description, xacro)
@@ -7,4 +7,5 @@
     <xacro:include
         filename="$(find s622_moveit_descriptions)/urdf/s622_moveit_descriptions.urdf.xacro" />
+    <!-- <xacro:property name="instantiate" value="false" /> -->
     <!-- ============ 左臂: base_link 在 (0.35, 0, 0), yaw=π ============ -->
     <xacro:s622_arm prefix="left_" attach_world="false" />

File: src/s622_moveit_descriptions/urdf/camera/camera.xacro (robot description, xacro)
@@ -6,5 +6,7 @@
   <xacro:include filename="$(find s622_moveit_descriptions)/urdf/camera/rgbd_split.gazebo.xacro" />
   <!-- ============================宏 1：相机本体 (URDF frames + mesh) ============================ -->
-  <xacro:macro name="camera_v0" params="parent *joint_origin">
+  <!-- use_camera_visual: true=真实 mesh(d435.dae)，false=简化几何体(渲染快，RViz 不卡)。
+       camera_link 本身必须保留（TF 树需要），只是 visual 形状不同。 -->
+  <xacro:macro name="camera_v0" params="parent use_camera_visual:=true *joint_origin">
     <xacro:sensor_d435
       parent="${parent}"
@@ -12,16 +14,19 @@
       use_nominal_extrinsics="true"
       add_plug="false"
-      use_mesh="true">
+      use_mesh="${use_camera_visual}">
       <xacro:insert_block name="joint_origin" />
     </xacro:sensor_d435>
   </xacro:macro>
   <!-- ============================宏 2：Gazebo 传感器 (分离 RGB + Depth) ============================ -->
+  <!-- 仿真性能：fps 60→20、960×540→640×480（对齐 robotarm），渲染负载降 ~7 倍 → RTF 大幅提升。
+       视觉伺服 50-100Hz 控制用锁定目标，20fps 检测足够。分辨率变化后 camera_info 自动更新，
+       visual_servo 的 use_adaptive_jacobian=true 运行时自适应，j_img_to_base 仅作 fallback。 -->
   <xacro:macro name="camera_gazebo_v0">
     <xacro:gazebo_rgbd_split
       name="camera"
-      fps="60"
+      fps="20"
       gz_topic_name="camera"
-      image_width="960"
-      image_height="540"
+      image_width="640"
+      image_height="480"
       h_fov="${82.4 * pi/180}"
       v_fov="${52.5 * pi/180}"

File: src/s622_moveit_descriptions/urdf/camera/rgbd_split.gazebo.xacro (robot description, xacro)
@@ -4,8 +4,8 @@
     params="
   name:=camera
-  fps:=30
+  fps:=20
   gz_topic_name:=camera
-  image_width:=960
-  image_height:=540
+  image_width:=640
+  image_height:=480
   h_fov
   v_fov

File: src/s622_moveit_descriptions/urdf/s622_moveit_descriptions.urdf.xacro (robot description, xacro)
@@ -7,5 +7,6 @@
     <xacro:arg name="prefix" default="" />
     <xacro:arg name="attach_world" default="true" />
-    <xacro:arg name="instantiate" default="true" />
+    <!-- <xacro:arg name="instantiate" default="true" /> -->
+         <xacro:arg name="instantiate" default="false" />
     <!-- ==================================================================
        Macro: s622_arm
