Commit message: feat(calib): M2 仿真环境搭建 —— 资产复制 + 右腕相机
- 复制 robotarm 资产：ros2_aruco（检测）、hand_eye_calibration（标定包）、
  aruco_5x5_250_id1 标定板模型
- camera.xacro：camera_v0/camera_gazebo_v0 支持 name 参数化（多相机不冲突）
- s622_dual_arm_gazebo.urdf.xacro：右臂 grasp_frame 加腕部相机 wrist_camera
  （GT=URDF 固定 origin 照 robotarm tool0 安装值；实验室仅 1 个腕部相机装右臂）
- 三个新包构建通过

File: src/gz_launch/config/s622_dual_arm_gazebo.urdf.xacro (robot description, xacro)
@@ -87,3 +87,12 @@
     </xacro:camera_v0>
     <xacro:camera_gazebo_v0 />
+    <!-- ============ [M2 标定] 右腕相机 (eye-in-hand GT) ============
+         2026-08-28：实验室仅 1 个腕部相机，装右臂 grasp_frame。
+         GT = URDF 固定 right_grasp_frame → wrist_camera 变换（origin 照 robotarm
+         tool0 安装值），标定后与求解结果比较（ground_truth_check_enabled=true）。 -->
+    <xacro:camera_v0 parent="right_grasp_frame" name="wrist_camera"
+                     use_camera_visual="$(arg include_camera_visual)">
+        <origin xyz="0 -0.05 -0.09" rpy="0 -1.57079632679 -1.57079632679" />
+    </xacro:camera_v0>
+    <xacro:camera_gazebo_v0 name="wrist_camera" />
 </robot>

File: src/s622_moveit_descriptions/urdf/camera/camera.xacro (robot description, xacro)
@@ -7,9 +7,11 @@
   <!-- ============================宏 1：相机本体 (URDF frames + mesh) ============================ -->
   <!-- use_camera_visual: true=真实 mesh(d435.dae)，false=简化几何体(渲染快，RViz 不卡)。
-       camera_link 本身必须保留（TF 树需要），只是 visual 形状不同。 -->
-  <xacro:macro name="camera_v0" params="parent use_camera_visual:=true *joint_origin">
+       camera_link 本身必须保留（TF 树需要），只是 visual 形状不同。
+       name: 相机实例名（默认 camera）。多相机（如腕部 wrist_camera）传不同 name，
+       生成 ${name}_link / ${name}_color_optical_frame 等唯一 frame。 -->
+  <xacro:macro name="camera_v0" params="parent name:=camera use_camera_visual:=true *joint_origin">
     <xacro:sensor_d435
       parent="${parent}"
-      name="camera"
+      name="${name}"
       use_nominal_extrinsics="true"
       add_plug="false"
@@ -21,10 +23,11 @@
   <!-- 仿真性能：fps 60→20、960×540→640×480（对齐 robotarm），渲染负载降 ~7 倍 → RTF 大幅提升。
        视觉伺服 50-100Hz 控制用锁定目标，20fps 检测足够。分辨率变化后 camera_info 自动更新，
-       visual_servo 的 use_adaptive_jacobian=true 运行时自适应，j_img_to_base 仅作 fallback。 -->
-  <xacro:macro name="camera_gazebo_v0">
+       visual_servo 的 use_adaptive_jacobian=true 运行时自适应，j_img_to_base 仅作 fallback。
+       name 必须与 camera_v0 的 name 一致。 -->
+  <xacro:macro name="camera_gazebo_v0" params="name:=camera">
     <xacro:gazebo_rgbd_split
-      name="camera"
+      name="${name}"
       fps="20"
-      gz_topic_name="camera"
+      gz_topic_name="${name}"
       image_width="640"
       image_height="480"
@@ -34,5 +37,5 @@
       max_depth="10.0"/>
     <!-- camera_link 材质 -->
-    <gazebo reference="camera_link">
+    <gazebo reference="${name}_link">
       <material>Gazebo/Grey</material>
     </gazebo>

Commit message: perf(calib): 桌面去腿（薄板）+ world 相机默认关闭 —— 减少 Gazebo 渲染
- table model.sdf：删除 4 条腿（collision+visual），只留 1.5×0.8 桌面薄板
  （模型已 static，不会坠落；所有用 table 的世界受益）
- s622_dual_arm_gazebo.urdf.xacro：world 俯视相机加 include_global_camera 参数
  默认 false（M2 标定用腕部 wrist_camera；M2.7 全局 eye-to-hand 再开）

File: src/gz_launch/config/s622_dual_arm_gazebo.urdf.xacro (robot description, xacro)
@@ -80,11 +80,17 @@
         initial_positions_file="$(find s622_moveit_config)/config/initial_positions.yaml"
         prefix="right_" />
-    <!-- ============ Camera 挂 world, 俯视 (0, 0, 0.75) ============ -->
+    <!-- ============ [M2] 全局俯视相机（默认关） ============
+         world 相机（0,0.5,0.9 俯视）是旧视觉伺服用；M2 标定用腕部 wrist_camera，
+         全局 eye-to-hand（M2.7）才需要它。默认关掉省一个 RGBD 渲染（Gazebo 卡因之一）。
+         需要时：include_global_camera:=true -->
+    <xacro:arg name="include_global_camera" default="false" />
     <xacro:include filename="$(find s622_moveit_descriptions)/urdf/camera/camera.xacro" />
-    <xacro:camera_v0 parent="world"
-                     use_camera_visual="$(arg include_camera_visual)">
-        <origin xyz="0 0.5 0.9" rpy="0 ${58*M_PI/180} ${-M_PI/2}" />
-    </xacro:camera_v0>
-    <xacro:camera_gazebo_v0 />
+    <xacro:if value="$(arg include_global_camera)">
+        <xacro:camera_v0 parent="world"
+                         use_camera_visual="$(arg include_camera_visual)">
+            <origin xyz="0 0.5 0.9" rpy="0 ${58*M_PI/180} ${-M_PI/2}" />
+        </xacro:camera_v0>
+        <xacro:camera_gazebo_v0 />
+    </xacro:if>
     <!-- ============ [M2 标定] 右腕相机 (eye-in-hand GT) ============
          2026-08-28：实验室仅 1 个腕部相机，装右臂 grasp_frame。

Commit message: perf(calib): wrist_camera 关 depth 渲染（标定只用 RGB，帧率 2.3Hz→提升）
实测 1280×720 RGB+depth 双传感器软件渲染仅 2.3Hz → 10 帧稳定窗口
凑不齐 → 全部 "insufficient stable marker frames"。关 depth 渲染减半。
gazebo_rgbd_split 加 enable_depth 参数；wrist_camera 传 false。

File: src/gz_launch/config/s622_dual_arm_gazebo.urdf.xacro (robot description, xacro)
@@ -101,4 +101,6 @@
         <origin xyz="0 -0.05 -0.09" rpy="0 -1.57079632679 -1.57079632679" />
     </xacro:camera_v0>
-    <xacro:camera_gazebo_v0 name="wrist_camera" />
+    <!-- [M2 标定] wrist_camera 只渲染 RGB（enable_depth=false）：标定只用 RGB，
+         关 depth 渲染减半 → 提升帧率（实测 1280×720 双传感器仅 2.3Hz → 稳定帧不足） -->
+    <xacro:camera_gazebo_v0 name="wrist_camera" enable_depth="false" />
 </robot>

File: src/s622_moveit_descriptions/urdf/camera/camera.xacro (robot description, xacro)
@@ -25,5 +25,5 @@
        visual_servo 的 use_adaptive_jacobian=true 运行时自适应，j_img_to_base 仅作 fallback。
        name 必须与 camera_v0 的 name 一致。 -->
-  <xacro:macro name="camera_gazebo_v0" params="name:=camera">
+  <xacro:macro name="camera_gazebo_v0" params="name:=camera enable_depth:=true">
     <xacro:gazebo_rgbd_split
       name="${name}"
@@ -35,5 +35,6 @@
       v_fov="${52.5 * pi/180}"
       min_depth="0.05"
-      max_depth="10.0"/>
+      max_depth="10.0"
+      enable_depth="${enable_depth}"/>
     <!-- camera_link 材质 -->
     <gazebo reference="${name}_link">

File: src/s622_moveit_descriptions/urdf/camera/rgbd_split.gazebo.xacro (robot description, xacro)
@@ -11,5 +11,6 @@
   v_fov
   min_depth:=0.05
-  max_depth:=10.0">
+  max_depth:=10.0
+  enable_depth:=true">  <!-- [M2 标定] enable_depth=false 只渲染 RGB（标定只用 RGB，关 depth 渲染减半 → 帧率提升） -->
     <xacro:property name="fx" value="${image_width * 0.5 / tan(h_fov * 0.5)}" />
     <xacro:property name="fy" value="${image_height * 0.5 / tan(v_fov * 0.5)}" />
@@ -56,5 +57,6 @@
       </sensor>
     </gazebo>
-    <!-- ===== Depth Sensor ===== -->
+    <!-- ===== Depth Sensor（[M2 标定] enable_depth=false 时关闭，减渲染负载） ===== -->
+    <xacro:if value="${enable_depth}">
     <gazebo reference="${name}_color_frame">
       <sensor name="${name}_depth" type="depth_camera">
@@ -96,4 +98,5 @@
       </sensor>
     </gazebo>
+    </xacro:if>
   </xacro:macro>
 </robot>

Commit message: feat(calib): M2.7 全局相机 eye-on-base 标定场景骨架（代码就绪，渲染待 GPU）
按 GPT 规划 M2.7 实施：
- xacro 三参数：include_global_camera（RGB-only 全局相机 (0,0.5,0.9)）/
  include_wrist_camera（标定期间关腕部提帧率）/ calibration_arm（left|right|none）
- 大号标定板：240mm 板 + 200mm marker（纹理 aruco_id1.png，DICT_5X5_250 id=1，
  cv2 实测 0.8~1.2m ≥90px），固定在 grasp_frame 上方平放，一次只挂一块
- s622_global_handeye_sim.launch.py：全局相机开+腕部关+aruco 检测+TF 发布
- s622_dual_arm.launch.py：透传参数 + wrist bridge 条件化 + spawn_robot 改
  OpaqueFunction（robot_description 含运行时 substitution）
- 左右两套 global_eye_on_base_{left,right}.yaml（eye_on_base/双臂 frame/
  marker 0.20/GT 校验开/输出分目录）
- derive_dual_base_from_camera.py：T_L_R_cam = T_L_C·inv(T_R_C) + URDF GT 比较
  （合成数据自测 0 误差）
- solver/evaluator/vision 零改动（复用 M2.2 eye_on_base 支持）
- 文档：M2.7_实施进度.md + 规划文档状态；附 GPT 规划原文两份
- xacro 三场景验证通过（right/left/default），launch 构造 OK

File: src/gz_launch/config/s622_dual_arm_gazebo.urdf.xacro (robot description, xacro)
@@ -83,5 +83,6 @@
          world 相机（0,0.5,0.9 俯视）是旧视觉伺服用；M2 标定用腕部 wrist_camera，
          全局 eye-to-hand（M2.7）才需要它。默认关掉省一个 RGBD 渲染（Gazebo 卡因之一）。
-         需要时：include_global_camera:=true -->
+         需要时：include_global_camera:=true
+         [M2.7] 标定只用 RGB → enable_depth=false 减半渲染负载 -->
     <xacro:arg name="include_global_camera" default="false" />
     <xacro:include filename="$(find s622_moveit_descriptions)/urdf/camera/camera.xacro" />
@@ -91,16 +92,95 @@
             <origin xyz="0 0.5 0.9" rpy="0 ${58*M_PI/180} ${-M_PI/2}" />
         </xacro:camera_v0>
-        <xacro:camera_gazebo_v0 />
+        <xacro:camera_gazebo_v0 enable_depth="false" />
+    </xacro:if>
+    <!-- ============ [M2.7] 全局 eye-to-hand 标定板（默认关） ============
+         大号 ArUco（板 160mm / marker 130mm，DICT_5X5_250 id=1，纹理 aruco_id1.png），
+         固定在指定臂的 grasp_frame 前方、板面朝 +x（全局相机在 (0,0.5,0.9) 俯视）。
+         一次只出现一块（calibration_arm:=left|right|none），避免两块同 ID 板同帧。
+         GT = 固定 joint 的 origin（可精确知道，但只用于最后 GT 验证，绝不喂 solver）。 -->
+    <xacro:arg name="calibration_arm" default="none" />
+    <xacro:property name="calib_arm" value="$(arg calibration_arm)" />
+    <xacro:if value="${calib_arm == 'left'}">
+        <link name="left_calibration_aruco">
+            <visual>
+                <origin xyz="0 0 0" rpy="0 0 0" />
+                <geometry>
+                    <box size="0.24 0.24 0.002" />
+                </geometry>
+            </visual>
+        </link>
+        <gazebo reference="left_calibration_aruco">
+            <visual>
+                <material>
+                    <ambient>1 1 1 1</ambient>
+                    <diffuse>1 1 1 1</diffuse>
+                    <specular>0 0 0 1</specular>
+                    <emissive>1 1 1 1</emissive>
+                    <pbr>
+                        <metal>
+                            <albedo_map>model://aruco_marker_1/materials/textures/aruco_id1.png</albedo_map>
+                            <emissive_map>model://aruco_marker_1/materials/textures/aruco_id1.png</emissive_map>
+                            <metalness>0.0</metalness>
+                            <roughness>1.0</roughness>
+                        </metal>
+                    </pbr>
+                </material>
+            </visual>
+        </gazebo>
+        <joint name="left_grasp_to_calibration_aruco" type="fixed">
+            <parent link="left_grasp_frame" />
+            <child link="left_calibration_aruco" />
+            <!-- 板面 +x：纹理正面朝全局相机方向（grasp_frame +x 朝前） -->
+            <origin xyz="0.05 0 0.08" rpy="1.5708 0 0" />
+        </joint>
+    </xacro:if>
+    <xacro:if value="${calib_arm == 'right'}">
+        <link name="right_calibration_aruco">
+            <visual>
+                <origin xyz="0 0 0" rpy="0 0 0" />
+                <geometry>
+                    <box size="0.24 0.24 0.002" />
+                </geometry>
+            </visual>
+        </link>
+        <gazebo reference="right_calibration_aruco">
+            <visual>
+                <material>
+                    <ambient>1 1 1 1</ambient>
+                    <diffuse>1 1 1 1</diffuse>
+                    <specular>0 0 0 1</specular>
+                    <emissive>1 1 1 1</emissive>
+                    <pbr>
+                        <metal>
+                            <albedo_map>model://aruco_marker_1/materials/textures/aruco_id1.png</albedo_map>
+                            <emissive_map>model://aruco_marker_1/materials/textures/aruco_id1.png</emissive_map>
+                            <metalness>0.0</metalness>
+                            <roughness>1.0</roughness>
+                        </metal>
+                    </pbr>
+                </material>
+            </visual>
+        </gazebo>
+        <joint name="right_grasp_to_calibration_aruco" type="fixed">
+            <parent link="right_grasp_frame" />
+            <child link="right_calibration_aruco" />
+            <origin xyz="0.05 0 0.08" rpy="1.5708 0 0" />
+        </joint>
     </xacro:if>
     <!-- ============ [M2 标定] 右腕相机 (eye-in-hand GT) ============
          2026-08-28：实验室仅 1 个腕部相机，装右臂 grasp_frame。
          GT = URDF 固定 right_grasp_frame → wrist_camera 变换（origin 照 robotarm
-         tool0 安装值），标定后与求解结果比较（ground_truth_check_enabled=true）。 -->
-    <xacro:camera_v0 parent="right_grasp_frame" name="wrist_camera"
-                     use_camera_visual="$(arg include_camera_visual)">
-        <origin xyz="0 -0.05 -0.09" rpy="0 -1.57079632679 -1.57079632679" />
-    </xacro:camera_v0>
-    <!-- [M2 标定] wrist_camera 只渲染 RGB（enable_depth=false）：标定只用 RGB，
-         关 depth 渲染减半 → 提升帧率（实测 1280×720 双传感器仅 2.3Hz → 稳定帧不足） -->
-    <xacro:camera_gazebo_v0 name="wrist_camera" enable_depth="false" />
+         tool0 安装值），标定后与求解结果比较（ground_truth_check_enabled=true）。
+         [M2.7] 全局 eye-to-hand 标定期间用 include_wrist_camera:=false 关掉它，
+         省一个 RGB 渲染 → 提升 Gazebo 帧率。 -->
+    <xacro:arg name="include_wrist_camera" default="true" />
+    <xacro:if value="$(arg include_wrist_camera)">
+        <xacro:camera_v0 parent="right_grasp_frame" name="wrist_camera"
+                         use_camera_visual="$(arg include_camera_visual)">
+            <origin xyz="0 -0.05 -0.09" rpy="0 -1.57079632679 -1.57079632679" />
+        </xacro:camera_v0>
+        <!-- [M2 标定] wrist_camera 只渲染 RGB（enable_depth=false）：标定只用 RGB，
+             关 depth 渲染减半 → 提升帧率（实测 1280×720 双传感器仅 2.3Hz → 稳定帧不足） -->
+        <xacro:camera_gazebo_v0 name="wrist_camera" enable_depth="false" />
+    </xacro:if>
 </robot>

Commit message: feat(calib): M2.7 双臂 Eye-on-Base 标定通过 — 修复集 + 3 次重复性统计
右臂 3 次(1.38/2.19/2.30mm)与左臂 3 次(0.40/2.55/1.38mm)独立采样均过 GT 门(≤3mm)；
T_L_R_cam 9 组合均值 4.93mm(>3mm,系统相关,详见记录文档)。

关键修复:
- launch: arm:= 参数生效(OpaqueFunction 设 M2_MODE)——此前 arm:=left 实际挂右板
- auto_collect: _move_arm 按 --arm 移动(原硬编码只动右臂); 助手三服务状态同步
- 内参: 渲染跟随 lens 使 focal_scale 无效 → marker_size_m 0.1988 补偿(仿真)
- 轴门 2->3mm 对齐 M2.7 验收④(每轴2mm 为 fairino EIH 遗留)
- 左臂 calib_board_visible 回填实测位姿(用户微调, 板居中 margin 189)

文档: M2.7_右臂EyeOnBase标定调试与通过_20260903.md(9章完整排查/统计),
intrinsics_bug_resolve 第11/12章复盘。

File: src/gz_launch/config/s622_dual_arm_gazebo.urdf.xacro (robot description, xacro)
@@ -132,5 +132,5 @@
             <child link="left_calibration_aruco" />
             <!-- 板面 +x：纹理正面朝全局相机方向（grasp_frame +x 朝前） -->
-            <origin xyz="0.05 0 0.08" rpy="1.5708 0 0" />
+            <origin xyz="0 0 0.13" rpy="1.5708 0 0" />
         </joint>
     </xacro:if>
@@ -165,5 +165,5 @@
             <parent link="right_grasp_frame" />
             <child link="right_calibration_aruco" />
-            <origin xyz="0.05 0 0.08" rpy="1.5708 0 0" />
+            <origin xyz="0 0 0.13" rpy="1.5708 0 0" />
         </joint>
     </xacro:if>

File: src/s622_moveit_descriptions/urdf/camera/camera.xacro (robot description, xacro)
@@ -24,6 +24,10 @@
        视觉伺服 50-100Hz 控制用锁定目标，20fps 检测足够。分辨率变化后 camera_info 自动更新，
        visual_servo 的 use_adaptive_jacobian=true 运行时自适应，j_img_to_base 仅作 fallback。
-       name 必须与 camera_v0 的 name 一致。 -->
-  <xacro:macro name="camera_gazebo_v0" params="name:=camera enable_depth:=true">
+       name 必须与 camera_v0 的 name 一致。
+       [M2.7 修正 2026-09-03 复盘] 曾用 focal_scale=0.9945 修正深度偏差——无效：
+       gz-sim 分离 camera 的渲染投影跟随 <lens> fx（≈0.9957×lens 常量偏移），
+       改 lens 会让渲染与 camera_info 一起变，solvePnP 深度自抵消。真正的独立杠杆是
+       标定配置里的 marker_size_m（见 global_eye_on_base_right.yaml 注释）。故还原 1.0。 -->
+  <xacro:macro name="camera_gazebo_v0" params="name:=camera enable_depth:=true focal_scale:=1.0">
     <xacro:gazebo_rgbd_split
       name="${name}"
@@ -34,4 +38,5 @@
       h_fov="${82.4 * pi/180}"
       v_fov="${52.5 * pi/180}"
+      focal_scale="${focal_scale}"
       min_depth="0.05"
       max_depth="10.0"

File: src/s622_moveit_descriptions/urdf/camera/rgbd_split.gazebo.xacro (robot description, xacro)
@@ -10,9 +10,20 @@
   h_fov
   v_fov
+  focal_scale:=1.0
   min_depth:=0.05
   max_depth:=10.0
   enable_depth:=true">  <!-- [M2 标定] enable_depth=false 只渲染 RGB（标定只用 RGB，关 depth 渲染减半 → 帧率提升） -->
-    <xacro:property name="fx" value="${image_width * 0.5 / tan(h_fov * 0.5)}" />
-    <xacro:property name="fy" value="${image_height * 0.5 / tan(v_fov * 0.5)}" />
+    <!-- [M2.7 修正复盘 2026-09-03] 曾用 focal_scale 乘到 fx/fy 修正深度偏差——无效。
+         实测结论（17/18 组样本 ×3 次数采 + 偏相关分析）：
+           - gz-sim 分离 camera 的渲染投影跟随 <lens> fx（render ≈ 0.9957×lens），
+             不是 <horizontal_fov>（resolve 文档实验 8 的结论混淆了两者同改）。
+           - 改 lens fx → 渲染与 camera_info 同向变化 → solvePnP 深度自抵消，
+             偏差 ~0.6% 依旧（GT 误差 4.5~5.3mm，3mm 门不过）。
+           - 偏差含 ~0.96px 系统性角点内缩（深度相关，斜率 ~1.7%/m）。
+         真正的独立杠杆 = 标定配置 marker_size_m（只改 solvePnP 假设，不动渲染），
+         取 0.1988（见 global_eye_on_base_right.yaml）。故 focal_scale 还原 1.0。
+         真机换 realsense-ros 无需任何补偿。 -->
+    <xacro:property name="fx" value="${image_width * 0.5 / tan(h_fov * 0.5) * focal_scale}" />
+    <xacro:property name="fy" value="${image_height * 0.5 / tan(v_fov * 0.5) * focal_scale}" />
     <xacro:property name="cx" value="${image_width * 0.5}" />
     <xacro:property name="cy" value="${image_height * 0.5}" />

Commit message: feat(m4): S1-P0 探针 — gz ApplyJointForce 可发力但会使 gz_ros2_control 位置伺服失效(力/速度命令互斥, 2/2 复现), S1-A 不成立; 插件默认关(安全) + 规划新增 §9/§10(Plan B 纯力控气动模型)

File: src/gz_launch/config/s622_dual_arm_gazebo.urdf.xacro (robot description, xacro)
@@ -3,4 +3,8 @@
     <xacro:property name="M_PI" value="3.14159265358979323846" />
     <xacro:arg name="instantiate" default="false" />   <!-- ← 加这行 -->
+    <!-- [M4_2 / S1] 是否给 finger 关节挂"夹持力"注入插件（ApplyJointForce）。
+         true=挂上（默认；插件在收到 cmd_force 前完全惰性）
+         false=完全不挂（A/B 对照用：排查插件是否干扰 position 控制） -->
+    <xacro:arg name="gripper_force_plugins" default="false" />
     <!-- 2026-08-25 对齐单臂/robotarm：include_camera_visual=false（默认）=
          简化几何体，RViz 不卡；true=真实 mesh（d435.dae） -->
@@ -26,4 +30,33 @@
             <render_engine>ogre2</render_engine>
         </plugin>
+        <!-- ==================================================================
+             [M4_2 / S1-P0] 夹爪"气压"等效：给 finger 关节注入常值夹持力。
+             真机：气动夹爪的夹持力由调压阀提供（软件只有开/关阀）；
+             仿真：gz_ros2_control 的 position 命令是"速度 ∝ 位置误差"的P型伺服，
+                   误差归零后夹持力=0（见 M4_0 §7.21）。故用 gz 原生插件在
+                   "被控对象层"补上这个力 —— 不改 ros2_control、不加控制器、
+                   不动真机任何文件。
+             接口：Double 消息 → /model/s622_dual_arm/joint/<joint>/cmd_force
+                   未收到消息前完全惰性（不影响既有行为）。
+             符号：沿关节轴。finger1 正=张开 → 夹持取负；finger2 反号。
+             ================================================================== -->
+        <xacro:if value="$(arg gripper_force_plugins)">
+        <plugin filename="ignition-gazebo-apply-joint-force-system"
+            name="gz::sim::systems::ApplyJointForce">
+            <joint_name>right_finger1_joint</joint_name>
+        </plugin>
+        <plugin filename="ignition-gazebo-apply-joint-force-system"
+            name="gz::sim::systems::ApplyJointForce">
+            <joint_name>right_finger2_joint</joint_name>
+        </plugin>
+        <plugin filename="ignition-gazebo-apply-joint-force-system"
+            name="gz::sim::systems::ApplyJointForce">
+            <joint_name>left_finger1_joint</joint_name>
+        </plugin>
+        <plugin filename="ignition-gazebo-apply-joint-force-system"
+            name="gz::sim::systems::ApplyJointForce">
+            <joint_name>left_finger2_joint</joint_name>
+        </plugin>
+        </xacro:if>
     </gazebo>
     <!-- ============ 引入 arm macro (M2.3 已 macro 化) ============ -->

Commit message: feat(m4): A'' 实现(关节限位=螺丝 + 直发close越界命令, 均默认关闭/真机零影响) + 双指自检与启动健康门工具; 实测阻塞: 初始位(全闭合0)与新限位自相矛盾导致 finger1 锁死(3/3), 记录三个解法

File: src/gz_launch/config/s622_dual_arm_gazebo.urdf.xacro (robot description, xacro)
@@ -7,4 +7,7 @@
          false=完全不挂（A/B 对照用：排查插件是否干扰 position 控制） -->
     <xacro:arg name="gripper_force_plugins" default="false" />
+    <!-- [M4_2 / A''] 夹爪"螺丝限位"（最小闭合间隙, m）。0.0=不启用(真机原始行程)。
+         仿真跑长条交接时由 launch 从环境变量 GRIPPER_STOP_GAP 传入，例如 0.029。 -->
+    <xacro:arg name="finger_stop_gap" default="0.0" />
     <!-- 2026-08-25 对齐单臂/robotarm：include_camera_visual=false（默认）=
          简化几何体，RViz 不卡；true=真实 mesh（d435.dae） -->
@@ -65,5 +68,5 @@
     <xacro:property name="instantiate" value="false" />
     <!-- ============ Left Arm: (0.35, 0, 0), yaw=π ============ -->
-    <xacro:s622_arm prefix="left_" attach_world="false" />
+    <xacro:s622_arm prefix="left_" attach_world="false" finger_stop_gap="$(arg finger_stop_gap)" />
     <joint name="left_mount_joint" type="fixed">
         <parent link="world" />
@@ -72,5 +75,5 @@
     </joint>
     <!-- ============ Right Arm: (-0.35, 0, 0), yaw=0 ============ -->
-    <xacro:s622_arm prefix="right_" attach_world="false" />
+    <xacro:s622_arm prefix="right_" attach_world="false" finger_stop_gap="$(arg finger_stop_gap)" />
     <joint name="right_mount_joint" type="fixed">
         <parent link="world" />

File: src/s622_moveit_descriptions/urdf/s622_moveit_descriptions.urdf.xacro (robot description, xacro)
@@ -9,9 +9,15 @@
     <!-- <xacro:arg name="instantiate" default="true" /> -->
          <xacro:arg name="instantiate" default="false" />
+    <!-- [M4_2 / A''] 夹爪"机械限位螺丝"等效：>0 时把两指行程下限收到 ±值/2
+         （即最小闭合间隙 = 该值）。默认 0.0 = 保留真机原始行程（真机零影响）。
+         只应由仿真侧（gz_launch 的 gazebo xacro）传入。 -->
+    <xacro:arg name="finger_stop_gap" default="0.0" />
     <!-- ==================================================================
        Macro: s622_arm
        双臂顶层需显式实例化两次, 各自不同 prefix + attach_world=false
        ================================================================== -->
-    <xacro:macro name="s622_arm" params="prefix:='' attach_world:=true">
+    <xacro:macro name="s622_arm" params="prefix:='' attach_world:=true finger_stop_gap:=0.0">
+        <!-- [M4_2 / A''] 限位半间隙；<=0 表示不启用额外限位 -->
+        <xacro:property name="finger_stop_half" value="${float(finger_stop_gap) * 0.5}" />
         <xacro:if value="${attach_world}">
             <link name="world" />
@@ -277,5 +283,5 @@
             <child link="${prefix}finger1" />
             <axis xyz="0.99996 0 -0.0087267" />
-            <limit lower="-1e-6" upper="0.0305" effort="150" velocity="3.2" />
+            <limit lower="${finger_stop_half if finger_stop_half > 0.0 else -1e-6}" upper="0.0305" effort="150" velocity="3.2" />
         </joint>
         <link name="${prefix}finger2">
@@ -307,5 +313,5 @@
             <child link="${prefix}finger2" />
             <axis xyz="0.99996 0 -0.0087267" />
-            <limit lower="-0.0305" upper="1e-6" effort="150" velocity="3.2" />
+            <limit lower="-0.0305" upper="${-finger_stop_half if finger_stop_half > 0.0 else 1e-6}" effort="150" velocity="3.2" />
         </joint>
         <!-- Grasp frame at the center of the gripper -->
@@ -362,5 +368,6 @@
        ================================================================== -->
     <xacro:if value="$(arg instantiate)">
-        <xacro:s622_arm prefix="$(arg prefix)" attach_world="$(arg attach_world)" />
+        <xacro:s622_arm prefix="$(arg prefix)" attach_world="$(arg attach_world)"
+            finger_stop_gap="$(arg finger_stop_gap)" />
     </xacro:if>
 </robot>
