Commit message: feat(m4): S3 物理限位块实现(默认关闭) + 实测: 起始状态落在挡块内导致穿模/MoveIt open 失败; 归档结构性结论(位置伺服+硬限位无法产生稳定夹持力)与修订路线 Plan B' 纯力控

File: src/gz_launch/config/s622_dual_arm_gazebo.urdf.xacro (robot description, xacro)
@@ -10,4 +10,7 @@
          仿真跑长条交接时由 launch 从环境变量 GRIPPER_STOP_GAP 传入，例如 0.029。 -->
     <xacro:arg name="finger_stop_gap" default="0.0" />
+    <!-- [M4_2 / S3] 夹爪"物理限位块"（推荐路线；默认关闭）。见下方 macro 注释。 -->
+    <xacro:arg name="gripper_stop_block" default="false" />
+    <xacro:arg name="gripper_stop_gap" default="0.028" />
     <!-- 2026-08-25 对齐单臂/robotarm：include_camera_visual=false（默认）=
          简化几何体，RViz 不卡；true=真实 mesh（d435.dae） -->
@@ -81,4 +84,45 @@
         <origin xyz="-0.35 0 0" rpy="0 0 0" />
     </joint>
+    <!-- ==================================================================
+         [M4_2 / S3] 夹爪"机械限位块"(等效真机拧螺丝定的最小闭合间隙)。
+         为什么需要: A'' 用关节限位做螺丝会与初始位(全闭合 0)冲突 -> finger1 被锁死
+         (M4_0/M4_2 §11 实测 3/3)。改用"物理挡块"：不动关节限位(初始位合法),
+         靠硬约束挡住指板继续合拢 -> 位置伺服误差永不归零 -> 持续夹持力。
+         几何(基于 §7.14/§7.17 标定, 单位: 相对 wrist3_link):
+           挡块宽(x) = 目标闭合间隙;  y = ±0.010(与指板等厚);  z ∈ [0.188, 0.204]
+           —— 放在【杆截面之后】: 杆占 wrist3 z ≈ [0.212, 0.242] (含 13° 倾斜余量),
+              挡块留 ~4mm 安全距离, 既不碰杆又能挡住指板内侧面。
+         默认关闭; 仿真跑长条交接时 GRIPPER_STOP_BLOCK=1 GRIPPER_STOP_GAP=0.028 启用。
+         ================================================================== -->
+    <xacro:macro name="gripper_stop_block" params="prefix gap:=0.028">
+        <link name="${prefix}gripper_stop">
+            <inertial>
+                <mass value="0.002" />
+                <inertia ixx="7e-08" ixy="0" ixz="0" iyy="7e-08" iyz="0" izz="7e-08" />
+            </inertial>
+            <collision name="collision">
+                <geometry>
+                    <box size="${gap} 0.020 0.016" />
+                </geometry>
+            </collision>
+            <visual name="visual">
+                <geometry>
+                    <box size="${gap} 0.020 0.016" />
+                </geometry>
+                <material name="">
+                    <color rgba="0.2 0.8 0.2 1.0" />
+                </material>
+            </visual>
+        </link>
+        <joint name="${prefix}gripper_stop_joint" type="fixed">
+            <parent link="${prefix}wrist3_link" />
+            <child link="${prefix}gripper_stop" />
+            <origin xyz="0 0 0.196" rpy="0 0 0" />
+        </joint>
+    </xacro:macro>
+    <xacro:if value="$(arg gripper_stop_block)">
+        <xacro:gripper_stop_block prefix="left_" gap="$(arg gripper_stop_gap)" />
+        <xacro:gripper_stop_block prefix="right_" gap="$(arg gripper_stop_gap)" />
+    </xacro:if>
     <!-- ============ Gripper 摩擦 (双臂各一份, 从 M2.1 前缀化) ============ -->
     <gazebo reference="left_finger1_joint">

Commit message: feat(C2.9a): Gazebo 125Hz position profile（QP 可在 Gazebo 里驱动双臂）
- s622_gazebo_ros2_control.xacro: 新增 arm_command_mode 参数(velocity|position),
  position 模式下臂暴露 position 接口 + position_proportional_gain=1.0
- s622_dual_arm_gazebo.urdf.xacro: 新增 arm_command_mode / controllers_yaml 参数
- dual_arm_qp_controller: 新增 Gazebo QP controllers yaml(+sweep 变体) 与
  独立精简 launch s622_dual_arm_qp.launch.py(不动原 JTC launch; profile 用环境变量选)
- 实测: 臂 16 position 接口/0 velocity; QP 控制器 active; sweep 关时 4s 零漂移,
  sweep 开时关节 p2p 0.018-0.069 rad; solver P99 0.10-0.23ms; 无故障
- ⚠️ 发现 1: gz_ros2_control 的 period 是合成值(恒 1/update_rate) -> PeriodMonitor
  在 Gazebo 永不触发; 控制器应自行差分 time 算实际周期
- ⚠️ 发现 2: Gazebo RTF≈0.46 -> 墙钟更新率 58Hz(仿真时间仍是 125Hz); Gazebo 不能
  验证墙钟实时余量, 只能验证单拍计算量与闭环动力学
- 遗留: C2.9b 互斥切换测试、Gazebo 里相对位姿误差量化

File: src/gz_launch/config/s622_dual_arm_gazebo.urdf.xacro (robot description, xacro)
@@ -16,4 +16,10 @@
          简化几何体，RViz 不卡；true=真实 mesh（d435.dae） -->
     <xacro:arg name="include_camera_visual" default="false" />
+    <!-- [C2.9a] arm command interface: velocity (JTC profile, default) or
+         position (QP profile, 125 Hz) -->
+    <xacro:arg name="arm_command_mode" default="velocity" />
+    <!-- [C2.9a] controllers yaml loaded by the gz_ros2_control plugin -->
+    <xacro:arg name="controllers_yaml"
+        default="$(find s622_moveit_config)/config/dual_arm_controllers.yaml" />
     <!-- ============ world 根 link ============ -->
     <link name="world" />
@@ -22,5 +28,5 @@
         <plugin filename="gz_ros2_control-system"
             name="gz_ros2_control::GazeboSimROS2ControlPlugin">
-            <parameters>$(find s622_moveit_config)/config/dual_arm_controllers.yaml</parameters>
+            <parameters>$(arg controllers_yaml)</parameters>
         </plugin>
         <plugin filename="gz-sim-joint-state-publisher-system"
@@ -155,9 +161,9 @@
         name="GazeboSimSystem"
         initial_positions_file="$(find s622_moveit_config)/config/initial_positions.yaml"
-        prefix="left_" />
+        prefix="left_" arm_command_mode="$(arg arm_command_mode)" />
     <xacro:s622_moveit_descriptions_ros2_control
         name="GazeboSimSystem"
         initial_positions_file="$(find s622_moveit_config)/config/initial_positions.yaml"
-        prefix="right_" />
+        prefix="right_" arm_command_mode="$(arg arm_command_mode)" />
     <!-- ============ [M2] 全局俯视相机（默认关） ============
          world 相机（0,0.5,0.9 俯视）是旧视觉伺服用；M2 标定用腕部 wrist_camera，

File: src/gz_launch/config/s622_gazebo_ros2_control.xacro (robot description, xacro)
@@ -3,5 +3,13 @@
     <!-- 增加 prefix 参数, 默认为空以保持 M1.7 兼容 -->
     <xacro:macro name="s622_moveit_descriptions_ros2_control"
-        params="name initial_positions_file prefix:=''">
+        params="name initial_positions_file prefix:='' arm_command_mode:='velocity'">
+        <!-- [C2.9a] arm command interface selectable: velocity (JTC profile) or
+             position (QP profile).  gz_ros2_control implements the position
+             interface as a P-type servo: velocity ~= gain * (target - current). -->
+        <xacro:property name="arm_cmd_iface"
+            value="${'position' if arm_command_mode == 'position' else 'velocity'}" />
+        <xacro:if value="${arm_command_mode == 'position'}">
+            <xacro:property name="arm_pos_gain" value="${1.0}" />
+        </xacro:if>
         <xacro:property name="initial_positions"
             value="${load_yaml(initial_positions_file)['initial_positions']}" />
@@ -12,5 +20,8 @@
             <!-- 6 个关节全部前缀化,同时 initial_positions 用无前缀 key 索引 -->
             <joint name="${prefix}j1">
-                <command_interface name="velocity" />
+                <command_interface name="${arm_cmd_iface}" />
+                <xacro:if value="${arm_command_mode == 'position'}">
+                    <param name="position_proportional_gain">${arm_pos_gain}</param>
+                </xacro:if>
                 <state_interface name="position">
                     <param name="initial_value">${initial_positions['j1']}</param>
@@ -19,5 +30,8 @@
             </joint>
             <joint name="${prefix}j2">
-                <command_interface name="velocity" />
+                <command_interface name="${arm_cmd_iface}" />
+                <xacro:if value="${arm_command_mode == 'position'}">
+                    <param name="position_proportional_gain">${arm_pos_gain}</param>
+                </xacro:if>
                 <state_interface name="position">
                     <param name="initial_value">${initial_positions['j2']}</param>
@@ -26,5 +40,8 @@
             </joint>
             <joint name="${prefix}j3">
-                <command_interface name="velocity" />
+                <command_interface name="${arm_cmd_iface}" />
+                <xacro:if value="${arm_command_mode == 'position'}">
+                    <param name="position_proportional_gain">${arm_pos_gain}</param>
+                </xacro:if>
                 <state_interface name="position">
                     <param name="initial_value">${initial_positions['j3']}</param>
@@ -33,5 +50,8 @@
             </joint>
             <joint name="${prefix}j4">
-                <command_interface name="velocity" />
+                <command_interface name="${arm_cmd_iface}" />
+                <xacro:if value="${arm_command_mode == 'position'}">
+                    <param name="position_proportional_gain">${arm_pos_gain}</param>
+                </xacro:if>
                 <state_interface name="position">
                     <param name="initial_value">${initial_positions['j4']}</param>
@@ -40,5 +60,8 @@
             </joint>
             <joint name="${prefix}j5">
-                <command_interface name="velocity" />
+                <command_interface name="${arm_cmd_iface}" />
+                <xacro:if value="${arm_command_mode == 'position'}">
+                    <param name="position_proportional_gain">${arm_pos_gain}</param>
+                </xacro:if>
                 <state_interface name="position">
                     <param name="initial_value">${initial_positions['j5']}</param>
@@ -47,5 +70,8 @@
             </joint>
             <joint name="${prefix}j6">
-                <command_interface name="velocity" />
+                <command_interface name="${arm_cmd_iface}" />
+                <xacro:if value="${arm_command_mode == 'position'}">
+                    <param name="position_proportional_gain">${arm_pos_gain}</param>
+                </xacro:if>
                 <state_interface name="position">
                     <param name="initial_value">${initial_positions['j6']}</param>

Commit message: Sync public from master: C2.9a Gazebo 125Hz position profile

File: src/gz_launch/config/s622_dual_arm_gazebo.urdf.xacro (robot description, xacro)
@@ -3,7 +3,23 @@
     <xacro:property name="M_PI" value="3.14159265358979323846" />
     <xacro:arg name="instantiate" default="false" />   <!-- ← 加这行 -->
+    <!-- [M4_2 / S1] 是否给 finger 关节挂"夹持力"注入插件（ApplyJointForce）。
+         true=挂上（默认；插件在收到 cmd_force 前完全惰性）
+         false=完全不挂（A/B 对照用：排查插件是否干扰 position 控制） -->
+    <xacro:arg name="gripper_force_plugins" default="false" />
+    <!-- [M4_2 / A''] 夹爪"螺丝限位"（最小闭合间隙, m）。0.0=不启用(真机原始行程)。
+         仿真跑长条交接时由 launch 从环境变量 GRIPPER_STOP_GAP 传入，例如 0.029。 -->
+    <xacro:arg name="finger_stop_gap" default="0.0" />
+    <!-- [M4_2 / S3] 夹爪"物理限位块"（推荐路线；默认关闭）。见下方 macro 注释。 -->
+    <xacro:arg name="gripper_stop_block" default="false" />
+    <xacro:arg name="gripper_stop_gap" default="0.028" />
     <!-- 2026-08-25 对齐单臂/robotarm：include_camera_visual=false（默认）=
          简化几何体，RViz 不卡；true=真实 mesh（d435.dae） -->
     <xacro:arg name="include_camera_visual" default="false" />
+    <!-- [C2.9a] arm command interface: velocity (JTC profile, default) or
+         position (QP profile, 125 Hz) -->
+    <xacro:arg name="arm_command_mode" default="velocity" />
+    <!-- [C2.9a] controllers yaml loaded by the gz_ros2_control plugin -->
+    <xacro:arg name="controllers_yaml"
+        default="$(find s622_moveit_config)/config/dual_arm_controllers.yaml" />
     <!-- ============ world 根 link ============ -->
     <link name="world" />
@@ -12,5 +28,5 @@
         <plugin filename="gz_ros2_control-system"
             name="gz_ros2_control::GazeboSimROS2ControlPlugin">
-            <parameters>$(find s622_moveit_config)/config/dual_arm_controllers.yaml</parameters>
+            <parameters>$(arg controllers_yaml)</parameters>
         </plugin>
         <plugin filename="gz-sim-joint-state-publisher-system"
@@ -26,4 +42,33 @@
             <render_engine>ogre2</render_engine>
         </plugin>
+        <!-- ==================================================================
+             [M4_2 / S1-P0] 夹爪"气压"等效：给 finger 关节注入常值夹持力。
+             真机：气动夹爪的夹持力由调压阀提供（软件只有开/关阀）；
+             仿真：gz_ros2_control 的 position 命令是"速度 ∝ 位置误差"的P型伺服，
+                   误差归零后夹持力=0（见 M4_0 §7.21）。故用 gz 原生插件在
+                   "被控对象层"补上这个力 —— 不改 ros2_control、不加控制器、
+                   不动真机任何文件。
+             接口：Double 消息 → /model/s622_dual_arm/joint/<joint>/cmd_force
+                   未收到消息前完全惰性（不影响既有行为）。
+             符号：沿关节轴。finger1 正=张开 → 夹持取负；finger2 反号。
+             ================================================================== -->
+        <xacro:if value="$(arg gripper_force_plugins)">
+        <plugin filename="ignition-gazebo-apply-joint-force-system"
+            name="gz::sim::systems::ApplyJointForce">
+            <joint_name>right_finger1_joint</joint_name>
+        </plugin>
+        <plugin filename="ignition-gazebo-apply-joint-force-system"
+            name="gz::sim::systems::ApplyJointForce">
+            <joint_name>right_finger2_joint</joint_name>
+        </plugin>
+        <plugin filename="ignition-gazebo-apply-joint-force-system"
+            name="gz::sim::systems::ApplyJointForce">
+            <joint_name>left_finger1_joint</joint_name>
+        </plugin>
+        <plugin filename="ignition-gazebo-apply-joint-force-system"
+            name="gz::sim::systems::ApplyJointForce">
+            <joint_name>left_finger2_joint</joint_name>
+        </plugin>
+        </xacro:if>
     </gazebo>
     <!-- ============ 引入 arm macro (M2.3 已 macro 化) ============ -->
@@ -32,5 +77,5 @@
     <xacro:property name="instantiate" value="false" />
     <!-- ============ Left Arm: (0.35, 0, 0), yaw=π ============ -->
-    <xacro:s622_arm prefix="left_" attach_world="false" />
+    <xacro:s622_arm prefix="left_" attach_world="false" finger_stop_gap="$(arg finger_stop_gap)" />
     <joint name="left_mount_joint" type="fixed">
         <parent link="world" />
@@ -39,5 +84,5 @@
     </joint>
     <!-- ============ Right Arm: (-0.35, 0, 0), yaw=0 ============ -->
-    <xacro:s622_arm prefix="right_" attach_world="false" />
+    <xacro:s622_arm prefix="right_" attach_world="false" finger_stop_gap="$(arg finger_stop_gap)" />
     <joint name="right_mount_joint" type="fixed">
         <parent link="world" />
@@ -45,4 +90,45 @@
         <origin xyz="-0.35 0 0" rpy="0 0 0" />
     </joint>
+    <!-- ==================================================================
+         [M4_2 / S3] 夹爪"机械限位块"(等效真机拧螺丝定的最小闭合间隙)。
+         为什么需要: A'' 用关节限位做螺丝会与初始位(全闭合 0)冲突 -> finger1 被锁死
+         (M4_0/M4_2 §11 实测 3/3)。改用"物理挡块"：不动关节限位(初始位合法),
+         靠硬约束挡住指板继续合拢 -> 位置伺服误差永不归零 -> 持续夹持力。
+         几何(基于 §7.14/§7.17 标定, 单位: 相对 wrist3_link):
+           挡块宽(x) = 目标闭合间隙;  y = ±0.010(与指板等厚);  z ∈ [0.188, 0.204]
+           —— 放在【杆截面之后】: 杆占 wrist3 z ≈ [0.212, 0.242] (含 13° 倾斜余量),
+              挡块留 ~4mm 安全距离, 既不碰杆又能挡住指板内侧面。
+         默认关闭; 仿真跑长条交接时 GRIPPER_STOP_BLOCK=1 GRIPPER_STOP_GAP=0.028 启用。
+         ================================================================== -->
+    <xacro:macro name="gripper_stop_block" params="prefix gap:=0.028">
+        <link name="${prefix}gripper_stop">
+            <inertial>
+                <mass value="0.002" />
+                <inertia ixx="7e-08" ixy="0" ixz="0" iyy="7e-08" iyz="0" izz="7e-08" />
+            </inertial>
+            <collision name="collision">
+                <geometry>
+                    <box size="${gap} 0.020 0.016" />
+                </geometry>
+            </collision>
+            <visual name="visual">
+                <geometry>
+                    <box size="${gap} 0.020 0.016" />
+                </geometry>
+                <material name="">
+                    <color rgba="0.2 0.8 0.2 1.0" />
+                </material>
+            </visual>
+        </link>
+        <joint name="${prefix}gripper_stop_joint" type="fixed">
+            <parent link="${prefix}wrist3_link" />
+            <child link="${prefix}gripper_stop" />
+            <origin xyz="0 0 0.196" rpy="0 0 0" />
+        </joint>
+    </xacro:macro>
+    <xacro:if value="$(arg gripper_stop_block)">
+        <xacro:gripper_stop_block prefix="left_" gap="$(arg gripper_stop_gap)" />
+        <xacro:gripper_stop_block prefix="right_" gap="$(arg gripper_stop_gap)" />
+    </xacro:if>
     <!-- ============ Gripper 摩擦 (双臂各一份, 从 M2.1 前缀化) ============ -->
     <gazebo reference="left_finger1_joint">
@@ -75,9 +161,9 @@
         name="GazeboSimSystem"
         initial_positions_file="$(find s622_moveit_config)/config/initial_positions.yaml"
-        prefix="left_" />
+        prefix="left_" arm_command_mode="$(arg arm_command_mode)" />
     <xacro:s622_moveit_descriptions_ros2_control
         name="GazeboSimSystem"
         initial_positions_file="$(find s622_moveit_config)/config/initial_positions.yaml"
-        prefix="right_" />
+        prefix="right_" arm_command_mode="$(arg arm_command_mode)" />
     <!-- ============ [M2] 全局俯视相机（默认关） ============
          world 相机（0,0.5,0.9 俯视）是旧视觉伺服用；M2 标定用腕部 wrist_camera，

Commit message: feat(C2.9b): profile 互斥测试 + Gazebo 相对位姿误差量化(含根因)
- check_profile_exclusive.sh: QP profile 下, 同关节 position JTC 与 velocity JTC
  都必须被拒绝 -> 3/3 通过(资源层互斥, 不靠约定)
- dual_arm_qp_monitor: 订阅 /joint_states, 用同一套运动学算 ^L T_R 的 RMS/max
- Gazebo 实测(sweep 0.06m/4s): 位置 RMS 42mm / max 60.4mm, 旋转 RMS 0.0007°
- 根因: gz_ros2_control 的 position_proportional_gain 固定 0.1(tau=10s!),
  三条配置途径(joint param / hardware param / 插件 yaml 节点参数)全部无效
  -> Gazebo position profile 只能验证接口/互斥/安全/CBF, 不能验证跟踪精度
- 保留 arm_position_gain 参数并注明当前无效, 避免重复踩坑

File: src/gz_launch/config/s622_dual_arm_gazebo.urdf.xacro (robot description, xacro)
@@ -19,4 +19,6 @@
          position (QP profile, 125 Hz) -->
     <xacro:arg name="arm_command_mode" default="velocity" />
+    <!-- gz position-servo gain [1/s] (only used when arm_command_mode=position) -->
+    <xacro:arg name="arm_position_gain" default="1.0" />
     <!-- [C2.9a] controllers yaml loaded by the gz_ros2_control plugin -->
     <xacro:arg name="controllers_yaml"
@@ -161,9 +163,11 @@
         name="GazeboSimSystem"
         initial_positions_file="$(find s622_moveit_config)/config/initial_positions.yaml"
-        prefix="left_" arm_command_mode="$(arg arm_command_mode)" />
+        prefix="left_" arm_command_mode="$(arg arm_command_mode)"
+        arm_position_gain="$(arg arm_position_gain)" />
     <xacro:s622_moveit_descriptions_ros2_control
         name="GazeboSimSystem"
         initial_positions_file="$(find s622_moveit_config)/config/initial_positions.yaml"
-        prefix="right_" arm_command_mode="$(arg arm_command_mode)" />
+        prefix="right_" arm_command_mode="$(arg arm_command_mode)"
+        arm_position_gain="$(arg arm_position_gain)" />
     <!-- ============ [M2] 全局俯视相机（默认关） ============
          world 相机（0,0.5,0.9 俯视）是旧视觉伺服用；M2 标定用腕部 wrist_camera，

File: src/gz_launch/config/s622_gazebo_ros2_control.xacro (robot description, xacro)
@@ -3,5 +3,5 @@
     <!-- 增加 prefix 参数, 默认为空以保持 M1.7 兼容 -->
     <xacro:macro name="s622_moveit_descriptions_ros2_control"
-        params="name initial_positions_file prefix:='' arm_command_mode:='velocity'">
+        params="name initial_positions_file prefix:='' arm_command_mode:='velocity' arm_position_gain:=1.0">
         <!-- [C2.9a] arm command interface selectable: velocity (JTC profile) or
              position (QP profile).  gz_ros2_control implements the position
@@ -9,7 +9,8 @@
         <xacro:property name="arm_cmd_iface"
             value="${'position' if arm_command_mode == 'position' else 'velocity'}" />
-        <xacro:if value="${arm_command_mode == 'position'}">
-            <xacro:property name="arm_pos_gain" value="${1.0}" />
-        </xacro:if>
+        <!-- gz_ros2_control position interface = P servo: v = gain*(q_des-q).
+             gain 1.0 => tau = 1 s (very slow); a realistic joint servo is
+             ~10-30 /s.  Configurable so the QP can be tuned. -->
+        <xacro:property name="arm_pos_gain" value="${float(arm_position_gain)}" />
         <xacro:property name="initial_positions"
             value="${load_yaml(initial_positions_file)['initial_positions']}" />
@@ -17,11 +18,14 @@
             <hardware>
                 <plugin>gz_ros2_control/GazeboSimSystem</plugin>
+                <!-- [C2.9] gz_ros2_control reads this from hardware_parameters
+                     (a per-JOINT <param> is silently ignored and the default
+                     0.1 is used => tau = 10 s!). -->
+                <xacro:if value="${arm_command_mode == 'position'}">
+                    <param name="position_proportional_gain">${arm_pos_gain}</param>
+                </xacro:if>
             </hardware>
             <!-- 6 个关节全部前缀化,同时 initial_positions 用无前缀 key 索引 -->
             <joint name="${prefix}j1">
                 <command_interface name="${arm_cmd_iface}" />
-                <xacro:if value="${arm_command_mode == 'position'}">
-                    <param name="position_proportional_gain">${arm_pos_gain}</param>
-                </xacro:if>
                 <state_interface name="position">
                     <param name="initial_value">${initial_positions['j1']}</param>
@@ -31,7 +35,4 @@
             <joint name="${prefix}j2">
                 <command_interface name="${arm_cmd_iface}" />
-                <xacro:if value="${arm_command_mode == 'position'}">
-                    <param name="position_proportional_gain">${arm_pos_gain}</param>
-                </xacro:if>
                 <state_interface name="position">
                     <param name="initial_value">${initial_positions['j2']}</param>
@@ -41,7 +42,4 @@
             <joint name="${prefix}j3">
                 <command_interface name="${arm_cmd_iface}" />
-                <xacro:if value="${arm_command_mode == 'position'}">
-                    <param name="position_proportional_gain">${arm_pos_gain}</param>
-                </xacro:if>
                 <state_interface name="position">
                     <param name="initial_value">${initial_positions['j3']}</param>
@@ -51,7 +49,4 @@
             <joint name="${prefix}j4">
                 <command_interface name="${arm_cmd_iface}" />
-                <xacro:if value="${arm_command_mode == 'position'}">
-                    <param name="position_proportional_gain">${arm_pos_gain}</param>
-                </xacro:if>
                 <state_interface name="position">
                     <param name="initial_value">${initial_positions['j4']}</param>
@@ -61,7 +56,4 @@
             <joint name="${prefix}j5">
                 <command_interface name="${arm_cmd_iface}" />
-                <xacro:if value="${arm_command_mode == 'position'}">
-                    <param name="position_proportional_gain">${arm_pos_gain}</param>
-                </xacro:if>
                 <state_interface name="position">
                     <param name="initial_value">${initial_positions['j5']}</param>
@@ -71,7 +63,4 @@
             <joint name="${prefix}j6">
                 <command_interface name="${arm_cmd_iface}" />
-                <xacro:if value="${arm_command_mode == 'position'}">
-                    <param name="position_proportional_gain">${arm_pos_gain}</param>
-                </xacro:if>
                 <state_interface name="position">
                     <param name="initial_value">${initial_positions['j6']}</param>
