Commit message: fix(hardware): 回滚至 8/27 原版 + cmdT 参数化（8/28 ServoJ 14 排查收尾）
- fairino_hardware_interface: 移除 ServoJ 统计/ServoMoveStart，恢复裸 ServoJ，
  新增 servoj_cmd_t 参数（默认 0.0016，对齐 robotarm 验证值）
- servoj_bare_test: 新增 14 诊断环形缓冲 + cmdT/no_close 参数
- s622_real_ros2_control.xacro / s622_real_motion_demo.launch.py:
  servoj_cmd_t 与 demo_max_velocity 参数化
- docs: 简历项目描述、双臂协同规划文档入库

File: src/s622_moveit_config/config/s622_real_ros2_control.xacro (robot description, xacro)
@@ -10,5 +10,5 @@
         - 状态接口：position（真机插件只导出 position state，read() 从 SDK 读真实角）
         ================================================================== -->
-    <xacro:macro name="s622_real_ros2_control" params="name prefix ip">
+    <xacro:macro name="s622_real_ros2_control" params="name prefix ip servoj_cmd_t:=0.0016">
         <ros2_control name="${name}" type="system">
             <hardware>
@@ -16,4 +16,6 @@
                 <param name="ip">${ip}</param>
                 <param name="prefix">${prefix}</param>
+                <!-- 2026-08-28：cmdT 参数化（默认 0.0016 = robotarm/8/27 验证值） -->
+                <param name="servoj_cmd_t">${servoj_cmd_t}</param>
             </hardware>
             <joint name="${prefix}j1">

Commit message: feat(hardware): ServoJ I/O 分层重构 Phase 1（设计文档 v2.1）
- write() 分离：只锁内拷贝 _latest_command，不再同步调 ServoJ（SDK 阻塞不传播到主循环）
- io_loop 独立线程：周期=cmdT（默认 0.008/125Hz，start-to-start），唯一 FRRobot 调用者
- 会话级 ServoMoveStart（on_activate，失败拒绝激活）/ ServoMoveEnd（io_loop 收尾）
- command-step velocity guard：per-joint |Δq|/cmdT ≤ v_limit[i]（默认 2.5 rad/s），
  超限或上次慢调用 → 发 last_sent 防跳变（不追赶 latest_command）
- send-interval health check + ServoJ 调用 watchdog（>20ms → latch fault）
- 第一次 rc!=0 即 latch fault，read/write 返回 ERROR（不再 14,14,14…）
- 反馈/finger SetDO 移入 io_loop；on_deactivate：shutdown→join→CloseRPC（joinable 必 join）
- real_controllers.yaml：update_rate 恢复 500（与 ServoJ 频率解耦）
- s622_real_ros2_control.xacro：cmdT 默认 0.008 + 新参数（v_limit/stall/feedback 阈值）

File: src/s622_moveit_config/config/s622_real_ros2_control.xacro (robot description, xacro)
@@ -10,5 +10,5 @@
         - 状态接口：position（真机插件只导出 position state，read() 从 SDK 读真实角）
         ================================================================== -->
-    <xacro:macro name="s622_real_ros2_control" params="name prefix ip servoj_cmd_t:=0.0016">
+    <xacro:macro name="s622_real_ros2_control" params="name prefix ip servoj_cmd_t:=0.008">
         <ros2_control name="${name}" type="system">
             <hardware>
@@ -16,6 +16,20 @@
                 <param name="ip">${ip}</param>
                 <param name="prefix">${prefix}</param>
-                <!-- 2026-08-28：cmdT 参数化（默认 0.0016 = robotarm/8/27 验证值） -->
+                <!-- 2026-08-28 分层重构（设计文档 v2.1 §8）：
+                     servoj_cmd_t           默认 0.008（125Hz，Phase1）；Phase2 测 0.004（250Hz）
+                     servo_v_limit_0..5     per-joint 等效速度上限（rad/s），建议 0.8×真机限速（J3 重点保护）
+                     servo_stall_warn_ms    10ms 慢调用警告
+                     servo_stall_fault_ms   20ms stall → fault
+                     feedback_stale_fault_ms 100ms 反馈过期 → fault -->
                 <param name="servoj_cmd_t">${servoj_cmd_t}</param>
+                <param name="servo_v_limit_0">2.5</param>
+                <param name="servo_v_limit_1">2.5</param>
+                <param name="servo_v_limit_2">2.5</param>
+                <param name="servo_v_limit_3">2.5</param>
+                <param name="servo_v_limit_4">2.5</param>
+                <param name="servo_v_limit_5">2.5</param>
+                <param name="servo_stall_warn_ms">10.0</param>
+                <param name="servo_stall_fault_ms">20.0</param>
+                <param name="feedback_stale_fault_ms">100.0</param>
             </hardware>
             <joint name="${prefix}j1">
